File: ljn-videoart-dumper.kicad_pcb (KiCad board)
At the start: 2 copper layers, 68.6 x 53.3 mm, 8 parts, among them J1 Power, J2 Digital/PWM, J3 Analog, J4 Digital/PWM

Commit message: Add connector
Parts:
- added J5: Video Art Edge, TE_AMP_5530843-3:CONN_5530843-3_TYC, F.Cu at (108.4, 77.9)
Other:
- board text added: "1"

Commit message: Fix pin numbering before it gets embarrassing
Parts:
- added U1: 74HC165, Package_DIP:DIP-16_W7.62mm_Socket_LongPads, F.Cu at (150.2, 65.1)
- moved J5 8.92 mm to (112.1, 86.0)
Routing:
- added copper zone on B.Cu, net GND

Commit message: Rearrangement
Parts:
- moved J5 43.2 mm to (155.2, 84.8), turned to 180 degrees
- moved U1 42.8 mm to (109.5, 78.4), turned to 90 degrees
Other:
- board text added: "Label Side This Way"
- board text added: "ljn video art dumper"
- board text added: "v0.1, leadedsolder.com"

Commit message: Final re-route
Parts:
- added R1: 0Ω, Resistor_THT:R_Axial_DIN0207_L6.3mm_D2.5mm_P10.16mm_Horizontal, F.Cu at (136.8, 53.0)
- added U2: 74HC595, Package_DIP:DIP-16_W7.62mm_Socket_LongPads, F.Cu at (151.4, 65.7)
- added U3: 74HC595, Package_DIP:DIP-16_W7.62mm_Socket_LongPads, F.Cu at (127.3, 53.6)
- moved U1 5.08 mm to (109.5, 73.3)
Routing:
- net /SCL/A5: track 0.00 -> 118.1 mm, vias 0 -> 2
- net /SDA/A4: track 0.00 -> 118.0 mm, vias 0 -> 2
- net +5V: track 0.00 -> 91.6 mm, vias 0 -> 3
- net /*3: track 0.00 -> 70.5 mm, vias 0 -> 2
- net /4: track 0.00 -> 65.4 mm, vias 0 -> 2
- net /12: track 0.00 -> 55.2 mm, vias 0 -> 3
- net /ROM_OE: track 0.00 -> 52.0 mm, vias 0 -> 3
- net /8: track 0.00 -> 51.6 mm, vias 0 -> 2
- net /2: track 0.00 -> 51.4 mm, vias 0 -> 2
- net /ROM_D0: track 0.00 -> 41.9 mm, vias 0 -> 4
- net GND: track 0.00 -> 40.5 mm, vias 0 -> 5
- net /ROM_A8: track 0.00 -> 40.5 mm, vias 0 -> 2
- net /ROM_D1: track 0.00 -> 36.8 mm, vias 0 -> 4
- net /ROM_A9: track 0.00 -> 36.1 mm
- net /ROM_A13: track 0.00 -> 35.9 mm
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- added copper zone on F.Cu, net +5V
