File: ljn-videoart-dumper.kicad_pcb (KiCad board)
At the start: 2 copper layers, 68.6 x 53.3 mm, 15 parts, among them J1 Power, J2 Digital/PWM, J3 Analog, J4 Digital/PWM, J5 Video Art Edge, U1 74HC165, U2 74HC595, U3 74HC595

Commit message: Short MR to 5V
Connections:
- U2 pad 10: unconnected-(U2-~{SRCLR}-Pad10) -> +5V
- U3 pad 10: unconnected-(U3-~{SRCLR}-Pad10) -> +5V
Routing:
- net +5V: track 85.3 -> 100.4 mm, vias 5 -> 8
Changed lines of the file:
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@@
   (net 63 "unconnected-(U1-~{Q7}-Pad7)")
   (net 64 "Net-(U2-QH')")
-  (net 65 "unconnected-(U2-~{SRCLR}-Pad10)")
-  (net 66 "unconnected-(U3-QG-Pad6)")
-  (net 67 "unconnected-(U3-QH-Pad7)")
-  (net 68 "unconnected-(U3-QH'-Pad9)")
-  (net 69 "unconnected-(U3-~{SRCLR}-Pad10)")
+  (net 65 "unconnected-(U3-QG-Pad6)")
+  (net 66 "unconnected-(U3-QH-Pad7)")
+  (net 67 "unconnected-(U3-QH'-Pad9)")
   (footprint "Connector_PinSocket_2.54mm:PinSocket_1x08_P2.54mm_Vertical" locked (layer "F.Cu")
     (at 127.94 97.46 90)
@@
       (net 59 "/ROM_A13") (pinfunction "QF") (pintype "tri_state"))
     (pad "6" thru_hole oval (at 0 12.7 270) (size 2.4 1.6) (drill 0.8) (layers "*.Cu" "*.Mask")
-      (net 66 "unconnected-(U3-QG-Pad6)") (pinfunction "QG") (pintype "tri_state+no_connect"))
+      (net 65 "unconnected-(U3-QG-Pad6)") (pinfunction "QG") (pintype "tri_state+no_connect"))
     (pad "7" thru_hole oval (at 0 15.24 270) (size 2.4 1.6) (drill 0.8) (layers "*.Cu" "*.Mask")
-      (net 67 "unconnected-(U3-QH-Pad7)") (pinfunction "QH") (pintype "tri_state+no_connect"))
+      (net 66 "unconnected-(U3-QH-Pad7)") (pinfunction "QH") (pintype "tri_state+no_connect"))
     (pad "8" thru_hole oval (at 0 17.78 270) (size 2.4 1.6) (drill 0.8) (layers "*.Cu" "*.Mask")
       (net 1 "GND") (pinfunction "GND") (pintype "power_in"))
     (pad "9" thru_hole oval (at 7.62 17.78 270) (size 2.4 1.6) (drill 0.8) (layers "*.Cu" "*.Mask")
-      (net 68 "unconnected-(U3-QH'-Pad9)") (pinfunction "QH'") (pintype "output+no_connect"))
+      (net 67 "unconnected-(U3-QH'-Pad9)") (pinfunction "QH'") (pintype "output+no_connect"))
     (pad "10" thru_hole oval (at 7.62 15.24 270) (size 2.4 1.6) (drill 0.8) (layers "*.Cu" "*.Mask")
-      (net 69 "unconnected-(U3-~{SRCLR}-Pad10)") (pinfunction "~{SRCLR}") (pintype "input+no_connect"))
+      (net 3 "+5V") (pinfunction "~{SRCLR}") (pintype "input"))
     (pad "11" thru_hole oval (at 7.62 12.7 270) (size 2.4 1.6) (drill 0.8) (layers "*.Cu" "*.Mask")
       (net 12 "/12") (pinfunction "SRCLK") (pintype "input"))
@@
       (net 64 "Net-(U2-QH')") (pinfunction "QH'") (pintype "output"))
     (pad "10" thru_hole oval (at 7.62 15.24 270) (size 2.4 1.6) (drill 0.8) (layers "*.Cu" "*.Mask")
-      (net 65 "unconnected-(U2-~{SRCLR}-Pad10)") (pinfunction "~{SRCLR}") (pintype "input+no_connect"))
+      (net 3 "+5V") (pinfunction "~{SRCLR}") (pintype "input"))
     (pad "11" thru_hole oval (at 7.62 12.7 270) (size 2.4 1.6) (drill 0.8) (layers "*.Cu" "*.Mask")
       (net 12 "/12") (pinfunction "SRCLK") (pintype "input"))
@@
   (segment (start 160.9901 73.3601) (end 160.96 73.33) (width 0.6) (layer "F.Cu") (net 3))
   (segment (start 159.69 87.935) (end 160.9901 86.6349) (width 0.6) (layer "F.Cu") (net 3))
+  (segment (start 117.145 61.265) (end 117.145 63.297) (width 0.25) (layer "F.Cu") (net 3))
+  (segment (start 114.478 65.583) (end 114.605 65.71) (width 0.25) (layer "F.Cu") (net 3))
+  (segment (start 114.478 63.424) (end 114.478 65.583) (width 0.25) (layer "F.Cu") (net 3))
   (segment (start 160.9901 86.6349) (end 160.9901 73.3601) (width 0.6) (layer "F.Cu") (net 3))
+  (segment (start 141.275 73.33) (end 138.608 75.997) (width 0.25) (layer "F.Cu") (net 3))
+  (segment (start 117.145 63.297) (end 117.272 63.424) (width 0.25) (layer "F.Cu") (net 3))
   (segment (start 134.925 71.285664) (end 134.925 75.235) (width 0.6) (layer "F.Cu") (net 3))
   (segment (start 114.605 65.71) (end 114.605 67.615) (width 0.6) (layer "F.Cu") (net 3))
+  (segment (start 138.608 75.997) (end 138.481 75.997) (width 0.25) (layer "F.Cu") (net 3))
   (via (at 134.925 61.265) (size 0.6) (drill 0.4) (layers "F.Cu" "B.Cu") (net 3))
+  (via (at 117.272 63.424) (size 0.6) (drill 0.4) (layers "F.Cu" "B.Cu") (net 3))
+  (via (at 138.481 75.997) (size 0.6) (drill 0.4) (layers "F.Cu" "B.Cu") (net 3))
+  (via (at 114.478 63.424) (size 0.6) (drill 0.4) (layers "F.Cu" "B.Cu") (net 3))
   (via (at 160.96 73.33) (size 0.6) (drill 0.4) (layers "F.Cu" "B.Cu") (net 3))
   (via (at 114.605 67.615) (size 0.6) (drill 0.4) (layers "F.Cu" "B.Cu") (net 3))
   (via (at 134.925 75.235) (size 0.6) (drill 0.4) (layers "F.Cu" "B.Cu") (net 3))
   (via (at 134.925 67.615) (size 0.6) (drill 0.4) (layers "F.Cu" "B.Cu") (net 3))
+  (segment (start 137.719 75.235) (end 134.925 75.235) (width 0.25) (layer "B.Cu") (net 3))
   (segment (start 114.77 67.45) (end 134.76 67.45) (width 0.6) (layer "B.Cu") (net 3))
   (segment (start 132.385 61.265) (end 134.925 61.265) (width 0.6) (layer "B.Cu") (net 3))
@@
   (segment (start 160.96 73.33) (end 156.515 73.33) (width 0.6) (layer "B.Cu") (net 3))
   (segment (start 114.605 67.615) (end 114.77 67.45) (width 0.6) (layer "B.Cu") (net 3))
+  (segment (start 117.272 63.424) (end 114.478 63.424) (width 0.25) (layer "B.Cu") (net 3))
   (segment (start 154.61 75.235) (end 156.515 73.33) (width 0.6) (layer "B.Cu") (net 3))
+  (segment (start 138.481 75.997) (end 137.719 75.235) (width 0.25) (layer "B.Cu") (net 3))
   (segment (start 134.925 75.235) (end 154.61 75.235) (width 0.6) (layer "B.Cu") (net 3))
   (segment (start 138.735 59.995) (end 136.195 59.995) (width 0.25) (layer "B.Cu") (net 3))
