File: ljn-videoart-dumper.kicad_sch (KiCad schematic)
At the start: 11 parts, among them J1 Power, J2 Digital/PWM, J3 Analog, J4 Digital/PWM, J5 Video Art Edge, U1 74HC165, U2 74HC595, U3 74HC595

Commit message: Short MR to 5V
Connections:
- net +5V: now also U2.10 (~{SRCLR}), U3.10 (~{SRCLR})
- no-connect marks 18 -> 16
Other:
- note added: "10/23: Oops, forgot to pull the reset pin up"
Changed lines of the file:
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@@
   (no_connect (at 120.015 79.375))
   (no_connect (at 132.715 79.375))
-  (no_connect (at 195.58 57.785))
   (no_connect (at 120.015 76.835))
   (no_connect (at 120.015 86.995))
   (no_connect (at 215.265 123.19))
-  (no_connect (at 194.945 115.57))
   (no_connect (at 34.29 31.75))
   (no_connect (at 120.015 84.455))
@@
     (stroke (width 0) (type solid))
   )
+  (wire (pts (xy 180.34 106.68) (xy 180.34 115.57))
+    (stroke (width 0) (type default))
+  )
   (wire (pts (xy 29.21 26.67) (xy 29.21 41.91))
     (stroke (width 0) (type solid))
@@
     (stroke (width 0) (type default))
   )
+  (wire (pts (xy 180.34 115.57) (xy 194.945 115.57))
+    (stroke (width 0) (type default))
+  )
   (wire (pts (xy 74.295 129.54) (xy 83.185 129.54))
     (stroke (width 0) (type default))
@@
   )
   (wire (pts (xy 142.24 76.835) (xy 142.24 64.77))
+    (stroke (width 0) (type default))
+  )
+  (wire (pts (xy 180.34 57.785) (xy 195.58 57.785))
+    (stroke (width 0) (type default))
+  )
+  (wire (pts (xy 180.34 43.815) (xy 180.34 57.785))
     (stroke (width 0) (type default))
   )
@@
   (text "TODO: Other, larger ROMs might use this as bank\nswitching but we have no idea where they go, or\neven if those ROMs exist"
     (at 220.98 129.54 0)
+    (effects (font (size 1.27 1.27)) (justify left bottom))
+  )
+  (text "10/23: Oops, forgot to pull the reset pin up" (at 153.035 34.925 0)
     (effects (font (size 1.27 1.27)) (justify left bottom))
   )
@@
         (path "/e63e39d7-6ac0-4ffd-8aa3-1841a4541b55"
           (reference "J4") (unit 1)
+        )
+      )
+    )
+  )
+  (symbol (lib_name "+5V_6") (lib_id "power:+5V") (at 180.34 106.68 0) (unit 1)
+    (in_bom yes) (on_board yes) (dnp no) (fields_autoplaced)
+    (property "Reference" "#PWR020" (at 180.34 110.49 0)
+      (effects (font (size 1.27 1.27)) hide)
+    )
+    (property "Value" "+5V" (at 180.34 101.6 0)
+      (effects (font (size 1.27 1.27)))
+    )
+    (property "Footprint" "" (at 180.34 106.68 0)
+      (effects (font (size 1.27 1.27)) hide)
+    )
+    (property "Datasheet" "" (at 180.34 106.68 0)
+      (effects (font (size 1.27 1.27)) hide)
+    )
+    (pin "1")
+    (instances
+      (project "ljn-videoart-dumper"
+        (path "/e63e39d7-6ac0-4ffd-8aa3-1841a4541b55"
+          (reference "#PWR020") (unit 1)
         )
       )
@@
         )
       )
+    )
+  )
+  (symbol (lib_name "+5V_7") (lib_id "power:+5V") (at 180.34 43.815 0) (unit 1)
+    (in_bom yes) (on_board yes) (dnp no) (fields_autoplaced)
+    (property "Reference" "#PWR021" (at 180.34 47.625 0)
+      (effects (font (size 1.27 1.27)) hide)
+    )
+    (property "Value" "+5V" (at 180.34 39.37 0)
+      (effects (font (size 1.27 1.27)))
+    )
+    (property "Footprint" "" (at 180.34 43.815 0)
+      (effects (font (size 1.27 1.27)) hide)
+    )
+    (property "Datasheet" "" (at 180.34 43.815 0)
+      (effects (font (size 1.27 1.27)) hide)
+    )
+    (pin "1")
+    (instances
+      (project "ljn-videoart-dumper"
+        (path "/e63e39d7-6ac0-4ffd-8aa3-1841a4541b55"
+          (reference "#PWR021") (unit 1)
+        )
+      )
